Commit message: Add mocap teleoperation and RM65 kinematics

File: assets/arm/RM65-6F.urdf (robot description, URDF)
Before this commit: robot RM65-6F, 7 links, 6 joints
Joints:
- joint joint_1: limit lower=-3.106 upper=3.106 effort=60 velocity=3.14 -> lower=-3.106686069 upper=3.106686069 effort=60 velocity=3.141592654
- joint joint_2: limit lower=-2.2689 upper=2.2689 effort=60 velocity=3.14 -> lower=-2.268928028 upper=2.268928028 effort=60 velocity=3.141592654
- joint joint_3: limit lower=-2.356 upper=2.356 effort=30 velocity=3.14 -> lower=-2.356194490 upper=2.356194490 effort=30 velocity=3.926990817
- joint joint_4: limit lower=-3.106 upper=3.106 effort=10 velocity=3.14 -> lower=-3.106686069 upper=3.106686069 effort=10 velocity=3.926990817
- joint joint_5: limit lower=-2.234 upper=2.234 effort=10 velocity=3.14 -> lower=-2.234021443 upper=2.234021443 effort=10 velocity=3.926990817
- joint joint_6: limit lower=-6.28 upper=6.28 effort=10 velocity=3.14 -> lower=-6.283185307 upper=6.283185307 effort=10 velocity=3.926990817

File: assets/scenes/rm65_dexhand_scene.urdf (robot description, URDF)
Before this commit: robot rm65_dexhand_table_scene, 59 links, 58 joints
Links:
- added link screwdriver_blue
- added link screwdriver_red
- link screwdriver_blue_handle: geometry collision cylinder length=0.16 radius=0.018; visual cylinder length=0.16 radius=0.018
- link screwdriver_blue_shaft: geometry collision cylinder length=0.2 radius=0.006; visual cylinder length=0.2 radius=0.006
- link screwdriver_red_handle: geometry collision cylinder length=0.16 radius=0.018; visual cylinder length=0.16 radius=0.018
- link screwdriver_red_shaft: geometry collision cylinder length=0.2 radius=0.006; visual cylinder length=0.2 radius=0.006
- link work_table_leg_bl: geometry collision box size=0.08 0.08 0.610; visual box size=0.08 0.08 0.610
- link work_table_leg_br: geometry collision box size=0.08 0.08 0.610; visual box size=0.08 0.08 0.610
- link work_table_leg_fl: geometry collision box size=0.08 0.08 0.610; visual box size=0.08 0.08 0.610
- link work_table_leg_fr: geometry collision box size=0.08 0.08 0.610; visual box size=0.08 0.08 0.610
Joints:
- removed joint world_to_screwdriver_blue_handle
- removed joint world_to_screwdriver_blue_shaft
- removed joint world_to_screwdriver_red_handle
- removed joint world_to_screwdriver_red_shaft
- added joint screwdriver_blue_to_screwdriver_blue_handle: type fixed, parent screwdriver_blue, child screwdriver_blue_handle, origin xyz=-0.040 0 0 rpy=0 1.5708 0
- added joint screwdriver_blue_to_screwdriver_blue_shaft: type fixed, parent screwdriver_blue, child screwdriver_blue_shaft, origin xyz=0.140 0 0 rpy=0 1.5708 0
- added joint screwdriver_red_to_screwdriver_red_handle: type fixed, parent screwdriver_red, child screwdriver_red_handle, origin xyz=-0.040 0 0 rpy=0 1.5708 0
- added joint screwdriver_red_to_screwdriver_red_shaft: type fixed, parent screwdriver_red, child screwdriver_red_shaft, origin xyz=0.140 0 0 rpy=0 1.5708 0
- added joint world_to_screwdriver_blue: type floating, parent world, child screwdriver_blue, origin xyz=0.12 -0.16 0.675 rpy=0 0 -0.800000
- added joint world_to_screwdriver_red: type floating, parent world, child screwdriver_red, origin xyz=-0.18 0.12 0.675 rpy=0 0 0.350000
- joint joint_1: limit lower=-3.106 upper=3.106 effort=60 velocity=3.14 -> lower=-3.106686069 upper=3.106686069 effort=60 velocity=3.141592654
- joint joint_2: limit lower=-2.2689 upper=2.2689 effort=60 velocity=3.14 -> lower=-2.268928028 upper=2.268928028 effort=60 velocity=3.141592654
- joint joint_3: limit lower=-2.356 upper=2.356 effort=30 velocity=3.14 -> lower=-2.356194490 upper=2.356194490 effort=30 velocity=3.926990817
- joint joint_4: limit lower=-3.106 upper=3.106 effort=10 velocity=3.14 -> lower=-3.106686069 upper=3.106686069 effort=10 velocity=3.926990817
- joint joint_5: limit lower=-2.234 upper=2.234 effort=10 velocity=3.14 -> lower=-2.234021443 upper=2.234021443 effort=10 velocity=3.926990817
- joint joint_6: limit lower=-6.28 upper=6.28 effort=10 velocity=3.14 -> lower=-6.283185307 upper=6.283185307 effort=10 velocity=3.926990817
- joint world_to_work_table_leg_bl: origin xyz=-0.27 0.35 0.23 rpy=0 0 0 -> xyz=-0.450 0.35 0.305 rpy=0 0 0
- joint world_to_work_table_leg_br: origin xyz=0.63 0.35 0.23 rpy=0 0 0 -> xyz=0.450 0.35 0.305 rpy=0 0 0
- joint world_to_work_table_leg_fl: origin xyz=-0.27 -0.35 0.23 rpy=0 0 0 -> xyz=-0.450 -0.35 0.305 rpy=0 0 0
- joint world_to_work_table_leg_fr: origin xyz=0.63 -0.35 0.23 rpy=0 0 0 -> xyz=0.450 -0.35 0.305 rpy=0 0 0
- joint world_to_work_table_top: origin xyz=0.18 0 0.48 rpy=0 0 0 -> xyz=0.0 0 0.630 rpy=0 0 0
