Commit message: 适配环境，调整摄像头位置

File: assets/scenes/rm65_dexhand_scene.urdf (robot description, URDF)
Before this commit: robot rm65_dexhand, 45 links, 44 joints
Links:
- added link robot_stand_leg_bl; collision box size=0.06 0.06 0.58; visual box size=0.06 0.06 0.58
- added link robot_stand_leg_br; collision box size=0.06 0.06 0.58; visual box size=0.06 0.06 0.58
- added link robot_stand_leg_fl; collision box size=0.06 0.06 0.58; visual box size=0.06 0.06 0.58
- added link robot_stand_leg_fr; collision box size=0.06 0.06 0.58; visual box size=0.06 0.06 0.58
- added link robot_stand_top; collision box size=0.70 0.55 0.04; visual box size=0.70 0.55 0.04
- added link screwdriver_blue_handle; collision cylinder length=0.18 radius=0.018; visual cylinder length=0.18 radius=0.018
- added link screwdriver_blue_shaft; collision cylinder length=0.16 radius=0.006; visual cylinder length=0.16 radius=0.006
- added link screwdriver_red_handle; collision cylinder length=0.18 radius=0.018; visual cylinder length=0.18 radius=0.018
- added link screwdriver_red_shaft; collision cylinder length=0.16 radius=0.006; visual cylinder length=0.16 radius=0.006
- added link work_table_leg_bl; collision box size=0.08 0.08 0.46; visual box size=0.08 0.08 0.46
- added link work_table_leg_br; collision box size=0.08 0.08 0.46; visual box size=0.08 0.08 0.46
- added link work_table_leg_fl; collision box size=0.08 0.08 0.46; visual box size=0.08 0.08 0.46
- added link work_table_leg_fr; collision box size=0.08 0.08 0.46; visual box size=0.08 0.08 0.46
- added link work_table_top; collision box size=1.0 0.8 0.04; visual box size=1.0 0.8 0.04
- link floor_link: geometry collision box size=12 12 0.02; visual box size=12 12 0.02
Joints:
- removed joint world_to_floor
- added joint world_to_floor_link: type fixed, parent world, child floor_link, origin xyz=0 0 -0.01 rpy=0 0 0
- added joint world_to_robot_stand_leg_bl: type fixed, parent world, child robot_stand_leg_bl, origin xyz=-0.98 0.22 0.29 rpy=0 0 0
- added joint world_to_robot_stand_leg_br: type fixed, parent world, child robot_stand_leg_br, origin xyz=-0.42 0.22 0.29 rpy=0 0 0
- added joint world_to_robot_stand_leg_fl: type fixed, parent world, child robot_stand_leg_fl, origin xyz=-0.98 -0.22 0.29 rpy=0 0 0
- added joint world_to_robot_stand_leg_fr: type fixed, parent world, child robot_stand_leg_fr, origin xyz=-0.42 -0.22 0.29 rpy=0 0 0
- added joint world_to_robot_stand_top: type fixed, parent world, child robot_stand_top, origin xyz=-0.7 0 0.58 rpy=0 0 0
- added joint world_to_screwdriver_blue_handle: type fixed, parent world, child screwdriver_blue_handle, origin xyz=0.35 -0.16 0.525 rpy=0 1.5708 0.8
- added joint world_to_screwdriver_blue_shaft: type fixed, parent world, child screwdriver_blue_shaft, origin xyz=0.49 -0.04 0.525 rpy=0 1.5708 0.8
- added joint world_to_screwdriver_red_handle: type fixed, parent world, child screwdriver_red_handle, origin xyz=-0.02 0.12 0.525 rpy=0 1.5708 0
- added joint world_to_screwdriver_red_shaft: type fixed, parent world, child screwdriver_red_shaft, origin xyz=0.16 0.12 0.525 rpy=0 1.5708 0
- added joint world_to_work_table_leg_bl: type fixed, parent world, child work_table_leg_bl, origin xyz=-0.27 0.35 0.23 rpy=0 0 0
- added joint world_to_work_table_leg_br: type fixed, parent world, child work_table_leg_br, origin xyz=0.63 0.35 0.23 rpy=0 0 0
- added joint world_to_work_table_leg_fl: type fixed, parent world, child work_table_leg_fl, origin xyz=-0.27 -0.35 0.23 rpy=0 0 0
- added joint world_to_work_table_leg_fr: type fixed, parent world, child work_table_leg_fr, origin xyz=0.63 -0.35 0.23 rpy=0 0 0
- added joint world_to_work_table_top: type fixed, parent world, child work_table_top, origin xyz=0.18 0 0.48 rpy=0 0 0
- joint world_to_base: origin xyz=0 0 0 rpy=0 0 0 -> xyz=0 0 0.02 rpy=0 0 0; parent world -> robot_stand_top
- joint world_to_camera_front: origin xyz=1.0 0 0.8 rpy=0 1.0472 1.5708 -> xyz=2.4 -2.2 1.2 rpy=0 1.0472 0.7854
- joint world_to_camera_side: origin xyz=0 1.0 0.8 rpy=1.0472 0 3.1416 -> xyz=0 3.0 1.4 rpy=1.0472 0 3.1416
- joint world_to_camera_top: origin xyz=0.4 0 1.5 rpy=0 0 0 -> xyz=0.3 0 3.0 rpy=0 0 0

Commit message: 适配硬件

File: assets/scenes/rm65_dexhand_scene.urdf (robot description, URDF)
Before this commit: robot rm65_dexhand_table_scene, 61 links, 60 joints
Links:
- removed link screwdriver_blue
- removed link screwdriver_blue_handle
- removed link screwdriver_blue_shaft
- link work_table_leg_bl: geometry collision box size=0.08 0.08 0.660; visual box size=0.08 0.08 0.660
- link work_table_leg_br: geometry collision box size=0.08 0.08 0.660; visual box size=0.08 0.08 0.660
- link work_table_leg_fl: geometry collision box size=0.08 0.08 0.660; visual box size=0.08 0.08 0.660
- link work_table_leg_fr: geometry collision box size=0.08 0.08 0.660; visual box size=0.08 0.08 0.660
Joints:
- removed joint screwdriver_blue_to_screwdriver_blue_handle
- removed joint screwdriver_blue_to_screwdriver_blue_shaft
- removed joint world_to_screwdriver_blue
- joint world_to_screwdriver_red: origin xyz=-0.18 0.12 0.675 rpy=0 0 0.350000 -> xyz=-0.08 -0.02 0.718 rpy=0 0 1.221730
- joint world_to_work_table_leg_bl: origin xyz=-0.450 0.35 0.305 rpy=0 0 0 -> xyz=-0.450 0.35 0.330 rpy=0 0 0
- joint world_to_work_table_leg_br: origin xyz=0.450 0.35 0.305 rpy=0 0 0 -> xyz=0.450 0.35 0.330 rpy=0 0 0
- joint world_to_work_table_leg_fl: origin xyz=-0.450 -0.35 0.305 rpy=0 0 0 -> xyz=-0.450 -0.35 0.330 rpy=0 0 0
- joint world_to_work_table_leg_fr: origin xyz=0.450 -0.35 0.305 rpy=0 0 0 -> xyz=0.450 -0.35 0.330 rpy=0 0 0
- joint world_to_work_table_top: origin xyz=0.0 0 0.630 rpy=0 0 0 -> xyz=0 0 0.680 rpy=0 0 0

Commit message: 保存下一功能测试前的稳定版本
验证：RM65解析IK 6项通过；Python compileall通过。
集成测试27项中22项通过、4项场景基线漂移失败、1项受EGL环境限制。

File: assets/scenes/rm65_dexhand_scene.urdf (robot description, URDF)
Before this commit: robot rm65_dexhand_table_scene, 58 links, 57 joints
Links:
- removed link robot_stand_leg_bl
- removed link robot_stand_leg_br
- removed link robot_stand_leg_fl
- removed link robot_stand_leg_fr
- added link dog_support_table_leg_bl; collision box size=0.08 0.08 1.127; visual box size=0.08 0.08 1.127
- added link dog_support_table_leg_br; collision box size=0.08 0.08 1.127; visual box size=0.08 0.08 1.127
- added link dog_support_table_leg_fl; collision box size=0.08 0.08 1.127; visual box size=0.08 0.08 1.127
- added link dog_support_table_leg_fr; collision box size=0.08 0.08 1.127; visual box size=0.08 0.08 1.127
- added link dog_support_table_top; collision box size=1.0 0.9 0.04; visual box size=1.0 0.9 0.04
- link robot_stand_top: geometry visual mesh filename=../dog/dog_visual_0.STL scale=0.00025 0.00025 0.00025; visual mesh filename=../dog/dog_visual_1.STL scale=0.00025 0.00025 0.00025
- link work_table_leg_bl: geometry collision box size=0.08 0.08 1.739; visual box size=0.08 0.08 1.739
- link work_table_leg_br: geometry collision box size=0.08 0.08 1.739; visual box size=0.08 0.08 1.739
- link work_table_leg_fl: geometry collision box size=0.08 0.08 1.739; visual box size=0.08 0.08 1.739
- link work_table_leg_fr: geometry collision box size=0.08 0.08 1.739; visual box size=0.08 0.08 1.739
Joints:
- removed joint world_to_robot_stand_leg_bl
- removed joint world_to_robot_stand_leg_br
- removed joint world_to_robot_stand_leg_fl
- removed joint world_to_robot_stand_leg_fr
- added joint world_to_dog_support_table_leg_bl: type fixed, parent world, child dog_support_table_leg_bl, origin xyz=-1.150 0.400 0.564 rpy=0 0 0
- added joint world_to_dog_support_table_leg_br: type fixed, parent world, child dog_support_table_leg_br, origin xyz=-0.250 0.400 0.564 rpy=0 0 0
- added joint world_to_dog_support_table_leg_fl: type fixed, parent world, child dog_support_table_leg_fl, origin xyz=-1.150 -0.400 0.564 rpy=0 0 0
- added joint world_to_dog_support_table_leg_fr: type fixed, parent world, child dog_support_table_leg_fr, origin xyz=-0.250 -0.400 0.564 rpy=0 0 0
- added joint world_to_dog_support_table_top: type fixed, parent world, child dog_support_table_top, origin xyz=-0.7 0.0 1.147 rpy=0 0 0
- joint world_to_robot_stand_top: origin xyz=-0.7 0 0.58 rpy=0 0 0 -> xyz=-0.7 0 1.65908 rpy=0 0 0
- joint world_to_screwdriver_red: origin xyz=-0.08 -0.02 0.718 rpy=0 0 1.221730 -> xyz=-0.08 0.12 1.797 rpy=0 0 1.221730
- joint world_to_work_table_leg_bl: origin xyz=-0.450 0.35 0.330 rpy=0 0 0 -> xyz=-0.450 0.35 0.870 rpy=0 0 0
- joint world_to_work_table_leg_br: origin xyz=0.450 0.35 0.330 rpy=0 0 0 -> xyz=0.450 0.35 0.870 rpy=0 0 0
- joint world_to_work_table_leg_fl: origin xyz=-0.450 -0.35 0.330 rpy=0 0 0 -> xyz=-0.450 -0.35 0.870 rpy=0 0 0
- joint world_to_work_table_leg_fr: origin xyz=0.450 -0.35 0.330 rpy=0 0 0 -> xyz=0.450 -0.35 0.870 rpy=0 0 0
- joint world_to_work_table_top: origin xyz=0 0 0.680 rpy=0 0 0 -> xyz=0 0 1.759 rpy=0 0 0
